File: PCB/EasyBLDCV1_DRV8305/DRV8305Breakout.kicad_sch (KiCad schematic)
At the start: 39 parts, among them Q1 CSD16556Q5B, Q2 CSD16556Q5B, Q3 CSD16556Q5B, Q4 CSD16556Q5B, Q5 CSD16556Q5B, Q6 CSD16556Q5B, U1 DRV83053PHP, U3 TPD4E05U06DQAR

Commit message: Fixed Naming Scheme
Parts:
- removed Q1, Q2, Q3, Q4, Q5, Q6: CSD16556Q5B, CSD16556Q5B:DNK0008A, symbol CSD16556Q5B:CSD16556Q5B
- removed U1: DRV83053PHP, DRV8305:PHP0048G_N, symbol DRV8305:DRV83053PHP
- removed U3: TPD4E05U06DQAR, TPD4E05U06DQAR:DQA0010A, symbol TPD4E05U06DQAR:TPD4E05U06DQAR
- added Q1, Q2, Q3, Q4, Q5, Q6: CSD16556Q5B, EasyBLDC:DNK0008A, symbol EasyBLDC:CSD16556Q5B
- added U1: DRV83053PHP, EasyBLDC:PHP0048G_N, symbol EasyBLDC:DRV83053PHP
- added U3: TPD4E05U06DQAR, EasyBLDC:DQA0010A, symbol EasyBLDC:TPD4E05U06DQAR
Connections:
- net 3.3V: now also U1.48 (VREG_VREF)
- net EN_GATE: now also U1.1 (EN_GATE)
- net GH_A: now also Q1.4 (G), U1.36 (GHA)
- net GH_B: now also Q3.4 (G), U1.29 (GHB)
- net GH_C: now also Q5.4 (G), U1.28 (GHC)
- net GL_A: now also Q2.4 (G), U1.33 (GLA)
- net GL_B: now also Q4.4 (G), U1.32 (GLB)
- net GL_C: now also Q6.4 (G), U1.25 (GLC)
- net GND: now also U1.14 (GND), U1.20 (SP3), U1.22 (SP2), U1.24 (SP1), U1.45 (GND), U1.49 (PAD), U3.3 (GND), U3.8 (GND)
- net INH_A: now also U1.2 (INH_A)
- net INH_B: now also U1.4 (INH_B)
- net INH_C: now also U1.6 (INH_C)
- net INL_A: now also U1.3 (INL_A)
- net INL_B: now also U1.5 (INL_B)
- net INL_C: now also U1.7 (INL_C)
- net ISEN_A: now also U1.16 (SO1)
- net ISEN_B: now also U1.17 (SO2)
- net ISEN_C: now also U1.18 (SO3)
- net MOT_A: now also Q1.1 (S), Q1.2 (S), Q1.3 (S), Q2.5 (D), Q2.6 (D), Q2.7 (D), Q2.8 (D), U1.35 (SHA)
- net MOT_B: now also Q3.1 (S), Q3.2 (S), Q3.3 (S), Q4.5 (D), Q4.6 (D), Q4.7 (D), Q4.8 (D), U1.30 (SHB)
- net MOT_C: now also Q5.1 (S), Q5.2 (S), Q5.3 (S), Q6.5 (D), Q6.6 (D), Q6.7 (D), Q6.8 (D), U1.27 (SHC)
- net PVDD: now also Q1.5 (D), Q1.6 (D), Q1.7 (D), Q1.8 (D), Q3.5 (D), Q3.6 (D), Q3.7 (D), Q3.8 (D), Q5.5 (D), Q5.6 (D), Q5.7 (D), Q5.8 (D), U1.41 (PVDD)
- net SCLK: now also U1.12 (SCLK)
- net SDI: now also U1.10 (SDI)
- net SDO: now also U1.11 (SDO)
- net SL_A: now also Q2.1 (S), Q2.2 (S), Q2.3 (S), U1.23 (SN1), U1.34 (SLA)
- net SL_B: now also Q4.1 (S), Q4.2 (S), Q4.3 (S), U1.21 (SN2), U1.31 (SLB)
- net SL_C: now also Q6.1 (S), Q6.2 (S), Q6.3 (S), U1.19 (SN3), U1.26 (SLC)
- net VSEN_A: now also U3.2 (D1-)
- net VSEN_B: now also U3.4 (D2+)
- net VSEN_C: now also U3.5 (D2-)
- net VSEN_PVDD: now also U3.1 (D1+)
- net WAKE: now also U1.47 (WAKE)
- net nFAULT: now also U1.8 (FAULT_N)
- net nSCS: now also U1.9 (SCS_N)
- net at R1.2: now also U1.13 (PWRGD)
- net at C1.2: now also U1.15 (AVDD)
- net at C17.1: now also U1.37 (VCP_LSD)
- net at C15.2: now also U1.38 (VCPH)
- net at C7.1: now also U1.39 (CP2H)
- net at C7.2: now also U1.40 (CP2L)
- net at C2.2: now also U1.42 (CP1L)
- net at C2.1: now also U1.43 (CP1H)
- net at R2.2: now also U1.44 (VDRAIN)
- net at C3.2: now also U1.46 (DVDD)

Commit message: Progress on MCU Breakout
Parts:
- PA1, PB1, PC1: footprint TestPoint:TestPoint_Pad_D3.0mm -> TestPoint:TestPoint_Pad_D2.0mm
Changed lines of the file:
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@@
 			)
 		)
-		(property "Footprint" "TestPoint:TestPoint_Pad_D3.0mm"
+		(property "Footprint" "TestPoint:TestPoint_Pad_D2.0mm"
 			(at 67.31 66.04 0)
 			(effects
@@
 			)
 		)
-		(property "Footprint" "TestPoint:TestPoint_Pad_D3.0mm"
+		(property "Footprint" "TestPoint:TestPoint_Pad_D2.0mm"
 			(at 137.16 146.05 0)
 			(effects
@@
 			)
 		)
-		(property "Footprint" "TestPoint:TestPoint_Pad_D3.0mm"
+		(property "Footprint" "TestPoint:TestPoint_Pad_D2.0mm"
 			(at 67.31 146.05 0)
 			(effects

Commit message: Updated Inductor and excluded tps from BOM
Parts:
- PA1, PB1, PC1: now left out of the parts list
Changed lines of the file:
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@@
 		(unit 1)
 		(exclude_from_sim no)
-		(in_bom yes)
+		(in_bom no)
 		(on_board yes)
 		(dnp no)
@@
 		(unit 1)
 		(exclude_from_sim no)
-		(in_bom yes)
+		(in_bom no)
 		(on_board yes)
 		(dnp no)
@@
 		(unit 1)
 		(exclude_from_sim no)
-		(in_bom yes)
-		(on_board yes)
-		(dnp no)
+		(in_bom no)
+		(on_board yes)
+		(dnp no)

Commit message: Fixed errors with silkscreen overlaping vias. Generated final gerbers.
Other:
- company: Buckley Boards  -> Peter Buckley Engineering
Changed lines of the file:
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@@
 		(date "2024-08-06")
 		(rev "1.0")
-		(company "Buckley Boards ")
+		(company "Peter Buckley Engineering")
 	)
 	(junction
