File: PCB/EasyBLDCV1_DRV8305/EasyBLDCV1_DRV8305.kicad_sch (KiCad schematic)
At the start: 0 parts

Commit message: Fixed errors with silkscreen overlaping vias. Generated final gerbers.
Other:
- company: Buckley Boards  -> Peter Buckley Engineering
Changed lines of the file:
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@@
 		(date "2024-08-06")
 		(rev "1.0")
-		(company "Buckley Boards ")
+		(company "Peter Buckley Engineering")
 	)
 	(sheet
