File: PCB/EasyBLDCV2_MCF8329/EasyBLDCV2_MCF8329.kicad_pcb (KiCad board)
At the start: 4 copper layers, 72.4 x 45.7 mm, 74 parts, among them J1 10159560-A00221RLF, J2 Conn_01x05_Pin, Q1 CSD17573Q5B, Q2 CSD17573Q5B, Q3 CSD17573Q5B, Q4 CSD17573Q5B, Q5 CSD17573Q5B, Q6 CSD17573Q5B, U1 MCF8329A1IREER

Commit message: Finished V2
Parts:
- moved C1 0.13 mm to (51.4, 66.5)
Routing:
- net PVDD: track 42.2 -> 52.0 mm, vias 85 -> 117
- net AVDD: track 51.5 -> 60.6 mm, vias 4 -> 6
- net FGOUT: track 17.4 -> 20.8 mm
- net GND: track 31.0 -> 32.6 mm, vias 124 -> 157
