File: PCB/EasyBLDCV4_STSPIN32F0A/TMS320F28027FBreakout_sch.kicad_sch (KiCad schematic)
At the start: 10 parts, among them U1 STSPIN32F0A

Commit message: Finished Schematic Assigned Footprints
Parts:
- added C12: 10u, Capacitor_SMD:C_0805_2012Metric, symbol Device:C_Small
- added C13, C15, C16, C17, C18: 100n, Capacitor_SMD:C_0402_1005Metric, symbol Device:C_Small
- added C14: 22u, Capacitor_SMD:C_0805_2012Metric, symbol Device:C_Small
- added D1, D2: D, Diode_SMD:D_0402_1005Metric, symbol Device:D
- added L1: 22u, Inductor_SMD:L_0805_2012Metric, symbol Device:L
- added R18: 10k, Resistor_SMD:R_0402_1005Metric, symbol Device:R_US
- added R19: 1k, Resistor_SMD:R_0402_1005Metric, symbol Device:R_US
- added TP1: TELEMETRY, TestPoint:TestPoint_Pad_D3.0mm, symbol Connector:TestPoint
- added TP2: TestPoint, TestPoint:TestPoint_Pad_D3.0mm, symbol Connector:TestPoint
- C19: renamed from C20; footprint (none) -> Capacitor_SMD:C_0402_1005Metric
- C20: renamed from C19; footprint (none) -> Capacitor_SMD:C_0402_1005Metric
- C21: renamed from C18; footprint (none) -> Capacitor_SMD:C_0402_1005Metric
- D3: renamed from D1; footprint LED_SMD:LED_0805_2012Metric -> LED_SMD:LED_0603_1608Metric
- D4: renamed from D2; footprint LED_SMD:LED_0805_2012Metric -> LED_SMD:LED_0603_1608Metric
- R20: renamed from R1; footprint (none) -> Resistor_SMD:R_0402_1005Metric
- R21: renamed from R20; value 2k -> 10k; footprint Resistor_SMD:R_0603_1608Metric -> Resistor_SMD:R_0201_0603Metric
- R22: renamed from R21; value 890 -> 2.2k; footprint Resistor_SMD:R_0603_1608Metric -> Resistor_SMD:R_0201_0603Metric
- R23: renamed from R2; footprint (none) -> Resistor_SMD:R_0402_1005Metric
- renumbered U1 to U2
Connections:
- net AVDD: now also U2.10 (VDDA), U2.48 (VDD), C14.1, C15.1, C16.1, D2.1 (K), L1.1
- net GND: now also U2.20 (TESTMODE), U2.44 (GND), U2.49 (EPAD), C12.1, C13.2, C14.2, C15.2, C16.2, C17.2, C18.1, D1.2 (A), R18.1
- net PVDD: now also U2.8 (VM), C17.1
- net VOLT_SENSE: now also U2.18 (PA7)
- net BEMF_B: now reaches U2.1 (OP2P)
- net at U2.13 (PA2): now also R19.2
- net CURRENT_SENSE: now reaches U2.16 (PA5)
- net OP1O: now reaches U2.17 (PA6)
- net OP1O: now also U2.21 (OP1O)
- net BEMF_COMMON: now reaches U2.2 (OP2N)
- net BEMF_COMMON: now also U2.22 (OP1N), U2.46 (OP3N)
- net BEMF_C: now reaches U2.23 (OP1P)
- net OP2O: now reaches U2.3 (OP2O)
- net OP2O: now also U2.4 (PF0)
- net SWDIO: now reaches U2.37 (PA13_SWD_IO)
- net SWCLK: now reaches U2.38 (PA14_SWD_CLK)
- net at U2.40 (PB6): now also TP1.1
- net at U2.41 (PB7): now also TP2.1
- net at U2.42 (BOOT0): now also R18.2
- net BEMF_A: now reaches U2.45 (OP3P)
- net OP3O: now reaches U2.47 (OP3O)
- net OP3O: now also U2.5 (PF1)
- net at U2.6 (VREG12): now also C12.2, C18.2
- net NRST: now reaches U2.7 (NRST)
- net NRST: now also C13.1
- net at U2.9 (SW): now also D1.1 (K), L1.2
- new net SIGNAL: D2.2 (A), R19.1
- no-connect marks 0 -> 8
Other:
- note added: "STSPIN32F0A"
- note added: "STSPIN32F0A Status"
- note removed: "MCF8329A Status"
- moved on the sheet: C19, C20, C21, D3, D4, R20, R21, R22, R23, U2

Commit message: Started Layout
Parts:
- U2: footprint STSPIN32F0A:IC_STSPIN32F0A -> EasyBLDC:IC_STSPIN32F0A
Changed lines of the file:
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@@
 			)
 		)
-		(property "Footprint" "STSPIN32F0A:IC_STSPIN32F0A"
+		(property "Footprint" "EasyBLDC:IC_STSPIN32F0A"
 			(at 97.79 118.11 0)
 			(effects

Commit message: Design finished, ready for review
Parts:
- TP1, TP2: footprint TestPoint:TestPoint_Pad_D3.0mm -> TestPoint:TestPoint_Pad_D1.5mm
Changed lines of the file:
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@@
 			)
 		)
-		(property "Footprint" "TestPoint:TestPoint_Pad_D3.0mm"
+		(property "Footprint" "TestPoint:TestPoint_Pad_D1.5mm"
 			(at 64.77 133.35 0)
 			(effects
@@
 			)
 		)
-		(property "Footprint" "TestPoint:TestPoint_Pad_D3.0mm"
+		(property "Footprint" "TestPoint:TestPoint_Pad_D1.5mm"
 			(at 64.77 138.43 0)
 			(effects

Commit message: updated some shit idk
Parts:
- D4: value GREEN -> RED
Changed lines of the file:
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@@
 			)
 		)
-		(property "Value" "GREEN"
+		(property "Value" "RED"
 			(at 226.06 129.8574 90)
 			(effects

Commit message: Changed out 0201 resistors, production version
Parts:
- R21, R22: footprint Resistor_SMD:R_0201_0603Metric -> Resistor_SMD:R_0402_1005Metric
Changed lines of the file:
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@@
 			)
 		)
-		(property "Footprint" "Resistor_SMD:R_0201_0603Metric"
+		(property "Footprint" "Resistor_SMD:R_0402_1005Metric"
 			(at 205.994 139.446 90)
 			(effects
@@
 			)
 		)
-		(property "Footprint" "Resistor_SMD:R_0201_0603Metric"
+		(property "Footprint" "Resistor_SMD:R_0402_1005Metric"
 			(at 221.234 139.446 90)
 			(effects
